Commit message: [add] gazebo launch file
tortoisebot.launchの実行でロボットモデルをGazeboで起動できるようになった．

File: DockerUser/catkin_ws/src/tortoisebot/src/urdf/tortoisebot.urdf (robot description, URDF)
Before this commit: robot tortoisebot, 1 links, 0 joints
Links:
- added link front_caster, mass 0.1; collision box size=0.1 0.1 0.3; visual box size=0.1 0.1 0.3
- added link front_wheel, mass 0.1; collision cylinder length=0.05 radius=0.035; visual cylinder length=0.05 radius=0.035
- added link left_wheel, mass 0.1; collision cylinder length=0.05 radius=0.035; visual cylinder length=0.05 radius=0.035
- added link right_wheel, mass 0.1; collision cylinder length=0.05 radius=0.035; visual cylinder length=0.05 radius=0.035
- link base_link: mass None -> 1.0; geometry collision box size=0.6 0.3 0.3; visual box size=0.6 0.3 0.3
Joints:
- added joint front_caster_joint: type continuous, parent base_link, child front_caster, origin xyz=0.3 0 0 rpy=0 0 0, axis 0 0 1
- added joint front_wheel_joint: type continuous, parent front_caster, child front_wheel, origin xyz=0.05 0 -.15 rpy=-1.5708 0 0, axis 0 0 1
- added joint left_wheel_joint: type continuous, parent base_link, child left_wheel, origin xyz=-0.2825 0.125 -.15 rpy=-1.5708 0 0, axis 0 0 1
- added joint right_wheel_joint: type continuous, parent base_link, child right_wheel, origin xyz=-0.2825 -0.125 -.15 rpy=-1.5708 0 0, axis 0 0 1

Commit message: [test] multiple robots
作業途中のため，未動作

File: DockerUser/catkin_ws/src/tortoisebot/src/urdf/tortoisebot.urdf (robot description, URDF)
Before this commit: robot tortoisebot, 6 links, 5 joints
Links:
- removed link front_wheel
- removed link hokuyo_link
- removed link left_wheel
- removed link right_wheel
- added link dummy
Joints:
- removed joint front_wheel_joint
- removed joint hokuyo_joint
- removed joint left_wheel_joint
- removed joint right_wheel_joint
- added joint dummy_joint: type fixed, parent dummy, child base_link
